File: PCB/APEX/v4/main.brd (EAGLE design)
At the start: 68.7 x 51.8 mm, 22 parts

Commit message: transfer changes to parent file
Parts:
- moved A1 29.5 mm to (58.4, 99.1)
- moved SIMISO 0.25 mm to (73.4, 67.3)
- turned TINYLHS to 270 degrees
Connections:
- net AIN+: now also TINYLHS.8
- net GND: now also TINYRHS.2, TINYRHS.8
- net RX: now also TINYLHS.5
- net SCL: now also TINYRHS.6
- net SDA: now also TINYRHS.7
- net TX: now also TINYLHS.6
- net VCC: now also TINYRHS.1
Routing:
- net VCC: track 20.0 -> 191.2 mm, vias 0 -> 1
- net GND: track 19.7 -> 145.7 mm, vias 0 -> 1
- net SCL: track 0.00 -> 76.0 mm
- net SDA: track 0.00 -> 72.3 mm
- net AIN+: track 0.00 -> 45.2 mm
- net SIMPOW: track 59.0 -> 60.5 mm
- net TX: track 5.46 -> 6.01 mm
- net RX: track 5.45 -> 6.00 mm
Other:
- board size 68.7 x 51.8 mm -> 76.2 x 52.7 mm
- board text added: "5V Top Right"
- board text added: "AIN+ AIN_ SD VCC GND"
- board text added: "AMP"
- board text added: "BARO"
- board text added: "BNO085"
- board text added: "BOOT P0 P1 RST MOSI CS"
- board text added: "GND"
- board text added: "GND 1PPS VCC RXI TXO WAKEUP"
- board text added: "GPS"
- board text added: "NET VCC RST RX TX GND"
- board text added: "RING DTR MIC+ MIC- SPK+ SPK-"
- board text added: "RX TX Unused AIN+"
- board text added: "SCL"
- board text added: "SCL SDA GND"
- board text added: "SDA"
- board text added: "SIM Isolation"
- board text added: "SIM800L"
- board text added: "Tiny 2040"
- board text added: "USB C Up"
- board text added: "VCC"
- board text added: "VCC 3V3 GND SCL SDA INT"
- board text added: "VCC 3V3 GND SCL SDA RST"
- board text added: "VCC 3V3 GND SCL SDO SDA CS"
- board text added: "VCC GND"

Commit message: send changes to parent design
Routing:
- net GND: track 145.7 -> 149.9 mm
- net SDA: track 72.3 -> 75.2 mm
- net SIMPOW: track 60.5 -> 61.8 mm
- added copper zone on layer 1, net GND
- added copper zone on layer 16, net GND
Other:
- outline, holes or cut-outs redrawn
- board text added: "APEX Comms"
- board text added: "APEX Sensor Board"
- board text added: "Altitude Record Team"
- board text added: "GND VCC SD AIN- AIN+"
- board text added: "Headers Soldered Upside Down"
- board text added: "Push Through This Way"
- board text added: "Shrey Bohra, Rohit Singh, Jason Hon, Akshat Tripathi, Harry Allcock Julian Ting, Nathanael Jenkins, Rohin Nayar, Tash Tanim, Kwan Yiu Tam"

Commit message: backport changes to parent design
Parts:
- moved SENS-SDA 17.8 mm to (73.7, 40.6)
- moved SENS-VCC 12.7 mm to (73.7, 29.2)
- moved SENS-SCL 7.62 mm to (73.7, 36.8)
- moved SENS-GND 2.54 mm to (73.7, 33.0)
- moved EXTGND 0.65 mm to (73.8, 60.3)
- moved SIMISO 0.51 mm to (73.9, 67.3), turned to 90 degrees
- moved EXTV+ 0.18 mm to (73.8, 57.3)
Connections:
- net SIMPOW: now also U$1.RST
Routing:
- net VCC: track 191.5 -> 1.54 mm, vias 1 -> 0
- net GND: track 149.9 -> 13.9 mm, vias 1 -> 0
- net AIN+: track 45.2 -> 59.5 mm
- net SCL: track 76.4 -> 72.3 mm
- net SDA: track 75.2 -> 71.2 mm, vias 0 -> 1
- net SIMPOW: track 61.8 -> 60.2 mm
- added copper zone on layer 1, net VCC
- removed copper zone on layer 1, net GND
Other:
- board size 76.2 x 52.7 mm -> 76.2 x 52.1 mm
- board text added: "+ -"
- board text added: "Lipo"
