File: PCB/APEX/v4/hackspace_con.brd (EAGLE design)
At the start: 73.7 x 26.7 mm, 13 parts

Commit message: flip amp
Parts:
- flipped JP2 to the bottom
Routing:
- net AIN+: track 59.0 -> 44.7 mm
- net SIMPOW: track 94.6 -> 89.2 mm
- net GND: track 30.2 -> 31.9 mm
Changed lines of the file:
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@@
 <board>
 <plain>
-<wire x1="49.53" y1="-55.88" x2="39.37" y2="-55.88" width="0.127" layer="21"/>
-<wire x1="39.37" y1="-55.88" x2="36.83" y2="-53.34" width="0.127" layer="21" curve="-90"/>
-<wire x1="36.83" y1="-53.34" x2="36.83" y2="-34.29" width="0.127" layer="21"/>
-<wire x1="36.83" y1="-34.29" x2="39.37" y2="-31.75" width="0.127" layer="21" curve="-90"/>
-<wire x1="39.37" y1="-31.75" x2="49.53" y2="-31.75" width="0.127" layer="21"/>
-<wire x1="49.53" y1="-31.75" x2="52.07" y2="-34.29" width="0.127" layer="21" curve="-90"/>
-<wire x1="52.07" y1="-34.29" x2="52.07" y2="-53.34" width="0.127" layer="21"/>
-<wire x1="52.07" y1="-53.34" x2="49.53" y2="-55.88" width="0.127" layer="21" curve="-90"/>
+<wire x1="39.37" y1="-55.88" x2="49.53" y2="-55.88" width="0.127" layer="22"/>
+<wire x1="49.53" y1="-55.88" x2="52.07" y2="-53.34" width="0.127" layer="22" curve="90"/>
+<wire x1="52.07" y1="-53.34" x2="52.07" y2="-34.29" width="0.127" layer="22"/>
+<wire x1="52.07" y1="-34.29" x2="49.53" y2="-31.75" width="0.127" layer="22" curve="90"/>
+<wire x1="49.53" y1="-31.75" x2="39.37" y2="-31.75" width="0.127" layer="22"/>
+<wire x1="39.37" y1="-31.75" x2="36.83" y2="-34.29" width="0.127" layer="22" curve="90"/>
+<wire x1="36.83" y1="-34.29" x2="36.83" y2="-53.34" width="0.127" layer="22"/>
+<wire x1="36.83" y1="-53.34" x2="39.37" y2="-55.88" width="0.127" layer="22" curve="90"/>
 <wire x1="-20.32" y1="-30.48" x2="-20.32" y2="-57.15" width="0.254" layer="20"/>
 <wire x1="-20.32" y1="-57.15" x2="53.34" y2="-57.15" width="0.254" layer="20"/>
@@
 <dimension x1="53.34" y1="-57.15" x2="53.34" y2="-30.48" x3="57.15" y3="-43.815" textsize="1.778" textratio="15" layer="49"/>
 <text x="60.96" y="-78.74" size="1.778" layer="21" font="vector" ratio="15">SIM</text>
-<text x="39.37" y="-43.18" size="1.778" layer="21" font="vector" ratio="15">AMP</text>
+<text x="49.53" y="-43.18" size="1.778" layer="22" font="vector" ratio="15" rot="MR0">AMP</text>
 <text x="71.12" y="-69.85" size="1.778" layer="22" font="vector" ratio="15" rot="MR0">2040</text>
 </plain>
@@
 <attribute name="VALUE" x="-13.335" y="-36.83" size="1.27" layer="27" rot="R90"/>
 </element>
-<element name="JP2" library="microbuilder" package="1X05_ROUND_70" value="" x="44.45" y="-52.832" smashed="yes" rot="R180">
-<attribute name="VALUE" x="50.8" y="-50.927" size="0.4064" layer="27" ratio="10" rot="R180"/>
+<element name="JP2" library="microbuilder" package="1X05_ROUND_70" value="" x="44.45" y="-52.832" smashed="yes" rot="MR180">
+<attribute name="VALUE" x="38.1" y="-50.927" size="0.4064" layer="28" ratio="10" rot="MR180"/>
 </element>
 </elements>
@@
 </polygon>
 <wire x1="-11.43" y1="-39.37" x2="-10.16" y2="-38.1" width="1.27" layer="16"/>
-<wire x1="41.91" y1="-52.07" x2="41.91" y2="-52.832" width="1.27" layer="16"/>
-<wire x1="41.91" y1="-52.832" x2="41.91" y2="-54.61" width="1.27" layer="16"/>
-<wire x1="49.53" y1="-50.8" x2="49.53" y2="-52.832" width="1.27" layer="16"/>
-<wire x1="49.53" y1="-52.832" x2="49.53" y2="-54.61" width="1.27" layer="16"/>
 <wire x1="12.868" y1="-50.696" x2="15.136" y2="-50.696" width="1.27" layer="16"/>
 <wire x1="15.136" y1="-50.696" x2="15.24" y2="-50.8" width="1.27" layer="16"/>
@@
 <wire x1="33.868" y1="-43.196" x2="31.766" y2="-43.196" width="1.27" layer="16"/>
 <wire x1="31.766" y1="-43.196" x2="31.75" y2="-43.18" width="1.27" layer="16"/>
+<wire x1="33.884" y1="-43.18" x2="34.29" y2="-43.18" width="1.27" layer="16"/>
+<wire x1="39.37" y1="-52.832" x2="39.37" y2="-50.8" width="1.27" layer="16"/>
+<wire x1="39.37" y1="-52.832" x2="38.862" y2="-53.34" width="1.27" layer="16"/>
+<wire x1="38.862" y1="-53.34" x2="38.1" y2="-53.34" width="1.27" layer="16"/>
+<wire x1="46.99" y1="-52.832" x2="46.99" y2="-49.53" width="1.27" layer="16"/>
 <wire x1="33.868" y1="-43.196" x2="33.884" y2="-43.18" width="1.27" layer="16"/>
-<wire x1="33.884" y1="-43.18" x2="34.29" y2="-43.18" width="1.27" layer="16"/>
+<wire x1="34.29" y1="-43.18" x2="35.56" y2="-43.18" width="1.27" layer="16"/>
 <wire x1="1.27" y1="-23.3" x2="-6.9" y2="-22.86" width="0" layer="19" extent="1-1"/>
 <wire x1="-6.9" y1="-7.62" x2="-6.9" y2="-22.86" width="0" layer="19" extent="1-1"/>
 <wire x1="-7.62" y1="-38.1" x2="-6.9" y2="-22.86" width="0" layer="19" extent="1-1"/>
-<wire x1="67.31" y1="-44.45" x2="49.53" y2="-50.8" width="0" layer="19" extent="16-16"/>
+<wire x1="11.43" y1="-50.8" x2="-7.62" y2="-53.34" width="0" layer="19" extent="16-16"/>
+<wire x1="46.99" y1="-52.832" x2="39.37" y2="-52.832" width="0" layer="19" extent="1-1"/>
+<wire x1="67.31" y1="-44.45" x2="46.99" y2="-49.53" width="0" layer="19" extent="16-16"/>
 </signal>
 <signal name="VCC">
@@
 <wire x1="17.724" y1="-40.696" x2="12.868" y2="-40.696" width="1.27" layer="16"/>
 <wire x1="12.868" y1="-40.696" x2="12.868" y2="-43.196" width="1.27" layer="16"/>
-<wire x1="-16.51" y1="-33.02" x2="17.78" y2="-33.02" width="1.27" layer="16"/>
-<wire x1="17.78" y1="-33.02" x2="19.05" y2="-33.02" width="1.27" layer="16"/>
-<wire x1="46.99" y1="-52.832" x2="46.99" y2="-50.8" width="1.27" layer="16"/>
-<wire x1="46.99" y1="-50.8" x2="45.72" y2="-49.53" width="1.27" layer="16"/>
-<wire x1="45.72" y1="-49.53" x2="43.18" y2="-49.53" width="1.27" layer="16"/>
-<wire x1="43.18" y1="-49.53" x2="41.91" y2="-48.26" width="1.27" layer="16"/>
-<wire x1="41.91" y1="-48.26" x2="41.91" y2="-36.83" width="1.27" layer="16"/>
-<wire x1="41.91" y1="-36.83" x2="39.37" y2="-34.29" width="1.27" layer="16"/>
-<wire x1="20.32" y1="-34.29" x2="19.05" y2="-33.02" width="1.27" layer="16"/>
-<wire x1="39.37" y1="-34.29" x2="20.32" y2="-34.29" width="1.27" layer="16"/>
+<wire x1="41.91" y1="-52.832" x2="41.91" y2="-49.53" width="1.27" layer="16"/>
+<wire x1="41.91" y1="-49.53" x2="40.64" y2="-48.26" width="1.27" layer="16"/>
+<wire x1="40.64" y1="-48.26" x2="39.37" y2="-48.26" width="1.27" layer="16"/>
+<wire x1="39.37" y1="-48.26" x2="38.1" y2="-46.99" width="1.27" layer="16"/>
+<wire x1="38.1" y1="-38.1" x2="35.56" y2="-35.56" width="1.27" layer="16"/>
+<wire x1="27.94" y1="-35.56" x2="25.4" y2="-33.02" width="1.27" layer="16"/>
+<wire x1="38.1" y1="-46.99" x2="38.1" y2="-38.1" width="1.27" layer="16"/>
+<wire x1="35.56" y1="-35.56" x2="27.94" y2="-35.56" width="1.27" layer="16"/>
+<wire x1="25.4" y1="-33.02" x2="17.78" y2="-33.02" width="1.27" layer="16"/>
+<wire x1="-16.51" y1="-33.02" x2="-16.002" y2="-32.512" width="1.016" layer="16"/>
+<wire x1="-5.588" y1="-32.512" x2="-5.08" y2="-33.02" width="1.016" layer="16"/>
+<wire x1="-16.002" y1="-32.512" x2="-5.588" y2="-32.512" width="1.016" layer="16"/>
+<wire x1="-5.08" y1="-33.02" x2="17.78" y2="-33.02" width="1.27" layer="16"/>
 </signal>
 <signal name="AIN+">
@@
 <contactref element="A1" pad="7"/>
 <contactref element="TINYLHS" pad="8"/>
-<wire x1="37.592" y1="-52.832" x2="36.83" y2="-52.07" width="1.27" layer="16"/>
-<wire x1="37.592" y1="-52.832" x2="39.37" y2="-52.832" width="1.27" layer="16"/>
-<wire x1="36.83" y1="-52.07" x2="36.83" y2="-39.37" width="1.27" layer="16"/>
-<wire x1="36.83" y1="-39.37" x2="35.56" y2="-38.1" width="1.27" layer="16"/>
-<wire x1="31.75" y1="-38.1" x2="29.21" y2="-40.64" width="1.27" layer="16"/>
-<wire x1="29.21" y1="-40.64" x2="29.21" y2="-53.34" width="1.27" layer="16"/>
-<wire x1="35.56" y1="-38.1" x2="31.75" y2="-38.1" width="1.27" layer="16"/>
-<wire x1="29.21" y1="-53.34" x2="7.62" y2="-53.34" width="1.27" layer="16"/>
+<wire x1="49.53" y1="-52.832" x2="49.53" y2="-54.61" width="1.27" layer="16"/>
+<wire x1="49.53" y1="-54.61" x2="48.895" y2="-55.245" width="1.27" layer="16"/>
+<wire x1="27.94" y1="-53.34" x2="7.62" y2="-53.34" width="1.27" layer="16"/>
+<wire x1="48.895" y1="-55.245" x2="29.845" y2="-55.245" width="1.27" layer="16"/>
+<wire x1="29.845" y1="-55.245" x2="27.94" y2="-53.34" width="1.27" layer="16"/>
 <wire x1="7.62" y1="-53.34" x2="9.44" y2="-22.86" width="0" layer="19" extent="1-1"/>
 </signal>

Commit message: Update hackspace_con.brd
Parts:
- moved EXTGND 20.7 mm to (47.0, -40.6)
Routing:
- net VCC: track 30.1 -> 33.9 mm
Changed lines of the file:
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@@
 <layer number="23" name="tOrigins" color="15" fill="1" visible="yes" active="yes"/>
 <layer number="24" name="bOrigins" color="15" fill="1" visible="yes" active="yes"/>
-<layer number="25" name="tNames" color="7" fill="1" visible="no" active="yes"/>
+<layer number="25" name="tNames" color="7" fill="1" visible="yes" active="yes"/>
 <layer number="26" name="bNames" color="7" fill="1" visible="no" active="yes"/>
 <layer number="27" name="tValues" color="7" fill="1" visible="no" active="yes"/>
@@
 <dimension x1="-20.32" y1="-57.15" x2="53.34" y2="-57.15" x3="16.51" y3="-60.96" textsize="1.778" textratio="15" layer="49"/>
 <dimension x1="53.34" y1="-57.15" x2="53.34" y2="-30.48" x3="57.15" y3="-43.815" textsize="1.778" textratio="15" layer="49"/>
-<text x="60.96" y="-78.74" size="1.778" layer="21" font="vector" ratio="15">SIM</text>
-<text x="49.53" y="-43.18" size="1.778" layer="22" font="vector" ratio="15" rot="MR0">AMP</text>
-<text x="71.12" y="-69.85" size="1.778" layer="22" font="vector" ratio="15" rot="MR0">2040</text>
+<text x="21.59" y="-48.26" size="1.778" layer="21" font="vector" ratio="15">SIM</text>
+<text x="43.18" y="-44.45" size="1.778" layer="21" font="vector" ratio="15">AMP</text>
+<text x="-2.54" y="-44.45" size="1.778" layer="21" font="vector" ratio="15">2040</text>
 </plain>
 <attributes>
@@
 <attribute name="VALUE" x="-17.78" y="-52.07" size="0.0254" layer="28" rot="MR180"/>
 </element>
-<element name="EXTGND" library="wirepad" library_urn="urn:adsk.eagle:library:412" package="SMD2,54-5,08" package3d_urn="urn:adsk.eagle:package:30841/1" value="" x="67.31" y="-44.45" smashed="yes" rot="MR0">
-<attribute name="NAME" x="68.81" y="-46.95" size="1.27" layer="26" rot="MR90"/>
-<attribute name="POPULARITY" value="21" x="67.31" y="-44.45" size="1.778" layer="28" font="vector" ratio="15" rot="MR0" display="off"/>
-<attribute name="VALUE" x="67.31" y="-44.45" size="0.0254" layer="28" rot="MR0"/>
+<element name="EXTGND" library="wirepad" library_urn="urn:adsk.eagle:library:412" package="SMD2,54-5,08" package3d_urn="urn:adsk.eagle:package:30841/1" value="" x="46.99" y="-40.64" smashed="yes" rot="MR0">
+<attribute name="NAME" x="48.49" y="-43.14" size="1.27" layer="26" rot="MR90"/>
+<attribute name="POPULARITY" value="21" x="46.99" y="-40.64" size="1.778" layer="28" font="vector" ratio="15" rot="MR0" display="off"/>
+<attribute name="VALUE" x="46.99" y="-40.64" size="0.0254" layer="28" rot="MR0"/>
 </element>
 <element name="BAT" library="adafruit" package="JST-PH-2-THM-RA" value="" x="-13.208" y="-44.323" smashed="yes" rot="R90">
@@
 <wire x1="33.868" y1="-43.196" x2="31.766" y2="-43.196" width="1.27" layer="16"/>
 <wire x1="31.766" y1="-43.196" x2="31.75" y2="-43.18" width="1.27" layer="16"/>
-<wire x1="33.884" y1="-43.18" x2="34.29" y2="-43.18" width="1.27" layer="16"/>
 <wire x1="39.37" y1="-52.832" x2="39.37" y2="-50.8" width="1.27" layer="16"/>
 <wire x1="39.37" y1="-52.832" x2="38.862" y2="-53.34" width="1.27" layer="16"/>
@@
 <wire x1="46.99" y1="-52.832" x2="46.99" y2="-49.53" width="1.27" layer="16"/>
 <wire x1="33.868" y1="-43.196" x2="33.884" y2="-43.18" width="1.27" layer="16"/>
-<wire x1="34.29" y1="-43.18" x2="35.56" y2="-43.18" width="1.27" layer="16"/>
+<wire x1="33.884" y1="-43.18" x2="35.56" y2="-43.18" width="1.27" layer="16"/>
 <wire x1="1.27" y1="-23.3" x2="-6.9" y2="-22.86" width="0" layer="19" extent="1-1"/>
 <wire x1="-6.9" y1="-7.62" x2="-6.9" y2="-22.86" width="0" layer="19" extent="1-1"/>
@@
 <wire x1="11.43" y1="-50.8" x2="-7.62" y2="-53.34" width="0" layer="19" extent="16-16"/>
 <wire x1="46.99" y1="-52.832" x2="39.37" y2="-52.832" width="0" layer="19" extent="1-1"/>
-<wire x1="67.31" y1="-44.45" x2="46.99" y2="-49.53" width="0" layer="19" extent="16-16"/>
+<wire x1="46.99" y1="-40.64" x2="46.99" y2="-49.53" width="0" layer="19" extent="16-16"/>
 </signal>
 <signal name="VCC">
@@
 <wire x1="-17.78" y1="-49.53" x2="-17.78" y2="-48.26" width="2.54" layer="16"/>
 <wire x1="-17.78" y1="-52.07" x2="-17.78" y2="-55.453" width="2.54" layer="16"/>
-<wire x1="-12.7" y1="-35.56" x2="-16.51" y2="-35.56" width="0" layer="19" extent="1-1"/>
+<wire x1="-16.51" y1="-35.56" x2="-12.7" y2="-35.56" width="1.27" layer="16"/>
 <wire x1="-6.9" y1="-5.08" x2="-7.62" y2="-35.56" width="0" layer="19" extent="1-1"/>
 </signal>

Commit message: dims
Routing:
- net AIN+: track 44.7 -> 20.3 mm
Changed lines of the file:
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@@
 <layer number="23" name="tOrigins" color="15" fill="1" visible="yes" active="yes"/>
 <layer number="24" name="bOrigins" color="15" fill="1" visible="yes" active="yes"/>
-<layer number="25" name="tNames" color="7" fill="1" visible="yes" active="yes"/>
+<layer number="25" name="tNames" color="7" fill="1" visible="no" active="yes"/>
 <layer number="26" name="bNames" color="7" fill="1" visible="no" active="yes"/>
 <layer number="27" name="tValues" color="7" fill="1" visible="no" active="yes"/>
@@
 <layer number="47" name="Measures" color="7" fill="1" visible="no" active="yes"/>
 <layer number="48" name="Document" color="7" fill="1" visible="no" active="yes"/>
-<layer number="49" name="Reference" color="7" fill="1" visible="no" active="yes"/>
+<layer number="49" name="Reference" color="7" fill="1" visible="yes" active="yes"/>
 <layer number="50" name="dxf" color="7" fill="1" visible="no" active="no"/>
 <layer number="51" name="tDocu" color="6" fill="1" visible="yes" active="yes"/>
@@
 <text x="43.18" y="-44.45" size="1.778" layer="21" font="vector" ratio="15">AMP</text>
 <text x="-2.54" y="-44.45" size="1.778" layer="21" font="vector" ratio="15">2040</text>
+<dimension x1="-20.32" y1="-30.48" x2="-20.32" y2="-57.15" x3="-22.86" y3="-43.815" textsize="1.778" textratio="15" layer="49"/>
 </plain>
 <attributes>
@@
 <wire x1="-6.9" y1="-7.62" x2="-6.9" y2="-22.86" width="0" layer="19" extent="1-1"/>
 <wire x1="-7.62" y1="-38.1" x2="-6.9" y2="-22.86" width="0" layer="19" extent="1-1"/>
-<wire x1="11.43" y1="-50.8" x2="-7.62" y2="-53.34" width="0" layer="19" extent="16-16"/>
-<wire x1="46.99" y1="-52.832" x2="39.37" y2="-52.832" width="0" layer="19" extent="1-1"/>
-<wire x1="46.99" y1="-40.64" x2="46.99" y2="-49.53" width="0" layer="19" extent="16-16"/>
 </signal>
 <signal name="VCC">
@@
 <contactref element="A1" pad="7"/>
 <contactref element="TINYLHS" pad="8"/>
-<wire x1="49.53" y1="-52.832" x2="49.53" y2="-54.61" width="1.27" layer="16"/>
-<wire x1="49.53" y1="-54.61" x2="48.895" y2="-55.245" width="1.27" layer="16"/>
 <wire x1="27.94" y1="-53.34" x2="7.62" y2="-53.34" width="1.27" layer="16"/>
-<wire x1="48.895" y1="-55.245" x2="29.845" y2="-55.245" width="1.27" layer="16"/>
-<wire x1="29.845" y1="-55.245" x2="27.94" y2="-53.34" width="1.27" layer="16"/>
-<wire x1="7.62" y1="-53.34" x2="9.44" y2="-22.86" width="0" layer="19" extent="1-1"/>
+<wire x1="49.53" y1="-52.832" x2="27.94" y2="-53.34" width="0" layer="19" extent="16-16"/>
+<wire x1="9.44" y1="-22.86" x2="7.62" y2="-53.34" width="0" layer="19" extent="1-1"/>
 </signal>
 <signal name="RX">
